Commit message: Pinza + cámara frontal + IMU + odom de encoders en el Summit XLS
- Pinza paralela (2 dedos prismáticos, solo abre/cierra) fija al frente +
  cámara encima, en urdf/gripper.urdf.xacro (macro summit_gripper, opt-in
  con gripper:=true).
- Control gz_ros2_control: <ros2_control> + plugin gz_ros2_control-system
  namespaceado por robot + config/gripper_controllers.yaml
  (JointTrajectoryController sobre los dedos).
- IMU del chasis (sensor type=imu, /summitN/imu) + sistema Imu en
  empty_arena.sdf. Odom de encoders del MecanumDrive expuesta en
  /summitN/encoder_odom (el /odom ground-truth queda intacto).
- sim_summit.launch.py: arg gripper -> xacro gripper:=true, spawner del
  gripper_controller y bridges de imu/encoder_odom/camera.
- display_gripper.launch.py: visor solo-RViz con sliders (sin Gazebo).
- comandos.txt y CLAUDE.md documentados.

Co-Authored-By: Claude Opus 4.8 <noreply@anthropic.com>

File: swarm_ws/src/summit_xl_description/robots/summit_xl_omni.urdf.xacro (robot description, xacro)
@@ -13,5 +13,7 @@
   <xacro:property name="ns" value="$(arg robot_ns)"/>
   <xacro:arg name="prefix" default=""/>
+  <xacro:arg name="gripper" default="false"/>
   <xacro:include filename="$(find summit_xl_description)/urdf/bases/summit_xls_base.urdf.xacro"/>
+  <xacro:include filename="$(find summit_xl_description)/urdf/gripper.urdf.xacro"/>
   <!-- Parámetros (de summit_xls.urdf.xacro / omni_wheel.urdf.xacro) -->
   <xacro:property name="wheel_offset_x" value="0.2225"/>
@@ -80,4 +82,23 @@
     <origin xyz="-${wheel_offset_x} -${wheel_offset_y} ${wheel_offset_z}" rpy="0 0 0"/>
   </xacro:mecanum_wheel>
+  <!-- Pinza paralela al frente (solo si gripper:=true) -->
+  <xacro:if value="$(arg gripper)">
+    <xacro:summit_gripper prefix="$(arg prefix)"/>
+    <!-- gz_ros2_control: arranca un controller_manager por robot que actua
+         sobre los dedos. Va en namespace ${ns} para alinearse con el
+         robot_state_publisher namespaceado (de donde el plugin lee el
+         <ros2_control> del robot_description) -> controller_manager en
+         /${ns}/controller_manager. El YAML usa claves comodin /** para casar
+         con cualquier namespace. -->
+    <gazebo>
+      <plugin filename="gz_ros2_control-system"
+              name="gz_ros2_control::GazeboSimROS2ControlPlugin">
+        <parameters>$(find summit_xl_description)/config/gripper_controllers.yaml</parameters>
+        <ros>
+          <namespace>${ns}</namespace>
+        </ros>
+      </plugin>
+    </gazebo>
+  </xacro:if>
   <!-- LiDAR 2D sobre la tapa del chasis -->
   <link name="$(arg prefix)lidar_link">
@@ -98,4 +119,16 @@
     <child  link="$(arg prefix)lidar_link"/>
     <origin xyz="0.25 0 0.43" rpy="0 0 0"/>
+  </joint>
+  <!-- IMU en el centro del chasis (sobre base_link). Frame ENU del sensor. -->
+  <link name="$(arg prefix)imu_link">
+    <inertial>
+      <mass value="0.01"/>
+      <inertia ixx="1e-6" ixy="0" ixz="0" iyy="1e-6" iyz="0" izz="1e-6"/>
+    </inertial>
+  </link>
+  <joint name="imu_joint" type="fixed">
+    <parent link="$(arg prefix)base_link"/>
+    <child  link="$(arg prefix)imu_link"/>
+    <origin xyz="0 0 0.05" rpy="0 0 0"/>
   </joint>
   <!-- ============ Gazebo Harmonic ============ -->
@@ -140,4 +173,17 @@
     </plugin>
   </gazebo>
+  <!-- IMU nativo Harmonic. Requiere el sistema Imu en el <world> (ya esta en
+       tugbot_warehouse.sdf y empty_arena.sdf). Publica gz.msgs.IMU. -->
+  <gazebo reference="$(arg prefix)imu_link">
+    <sensor name="imu" type="imu">
+      <topic>/model/${ns}/imu</topic>
+      <gz_frame_id>${ns}/imu_link</gz_frame_id>
+      <update_rate>100</update_rate>
+      <always_on>1</always_on>
+      <imu>
+        <enable_orientation>true</enable_orientation>
+      </imu>
+    </sensor>
+  </gazebo>
   <gazebo reference="$(arg prefix)lidar_link">
     <sensor name="lidar" type="gpu_lidar">

Commit message: Basura en poses aleatorias con semilla reproducible
Las basuras dejan de estar hardcodeadas en el mundo y se generan con poses
aleatorias sembradas (rejection sampling), inyectadas en el <world> al
lanzar. Se inyectan (no se spawnean sueltas) porque los DetachableJoint del
gripper se enlazan a los modelos al CARGAR el robot: la basura debe existir
antes de spawnear el robot o el joint no se forma.

- sim_summit.launch.py: args n_trash (def 6) y seed (def 42, -1=aleatorio).
  _trash_poses() con rejection sampling en la zona norte (x[-6,6] y[13,23]),
  separando basuras entre si y de los spawns de los robots. Inyecta los
  modelos antes de </world> en /tmp/swarm_summit/<world>_gen.sdf. Pasa la
  lista de nombres (trash_0..N-1) al xacro y al detach inicial.
- gripper.urdf.xacro + summit_xl_omni.urdf.xacro: trash_list es ahora
  parametro del macro/arg; genera un DetachableJoint por basura segun los
  nombres del launch (vacio = ninguno).
- tugbot_warehouse.sdf: quitadas las 6 basuras hardcodeadas (plantilla).

Validado en vivo (headless, 1 robot, n_trash=6 seed=42): 6 basuras
inyectadas y cargadas en sus poses, detach inicial OK (no soldadas al mover
el robot), semilla reproducible (42==42, 42!=7), xacro genera los joints.

Co-Authored-By: Claude Opus 4.8 <noreply@anthropic.com>

File: swarm_ws/src/summit_xl_description/robots/summit_xl_omni.urdf.xacro (robot description, xacro)
@@ -14,4 +14,8 @@
   <xacro:arg name="prefix" default=""/>
   <xacro:arg name="gripper" default="false"/>
+  <!-- Nombres de las basuras (separados por espacio) para los DetachableJoint
+       del gripper. Los pasa el launch; deben coincidir con los modelos del
+       mundo. Vacío = sin DetachableJoint. -->
+  <xacro:arg name="trash_list" default=""/>
   <xacro:include filename="$(find summit_xl_description)/urdf/bases/summit_xls_base.urdf.xacro"/>
   <xacro:include filename="$(find summit_xl_description)/urdf/gripper.urdf.xacro"/>
@@ -84,5 +88,5 @@
   <!-- Pinza paralela al frente (solo si gripper:=true) -->
   <xacro:if value="$(arg gripper)">
-    <xacro:summit_gripper prefix="$(arg prefix)"/>
+    <xacro:summit_gripper prefix="$(arg prefix)" trash_list="$(arg trash_list)"/>
     <!-- gz_ros2_control: arranca un controller_manager por robot que actua
          sobre los dedos. Va en namespace ${ns} para alinearse con el

File: swarm_ws/src/summit_xl_description/urdf/gripper.urdf.xacro (robot description, xacro)
@@ -13,5 +13,5 @@
        en una fase posterior. Para verlo moverse en RViz basta el
        joint_state_publisher_gui (sliders sobre estos 2 joints). -->
-  <xacro:macro name="summit_gripper" params="prefix:=''">
+  <xacro:macro name="summit_gripper" params="prefix:='' trash_list:=''">
     <material name="gripper_dark"><color rgba="0.15 0.15 0.18 1"/></material>
     <material name="gripper_gray"><color rgba="0.5 0.5 0.55 1"/></material>
@@ -96,7 +96,7 @@
          'release'. parent_link = base_footprint (la palma se fusiona en el
          root al convertir URDF->SDF). child_link = 'link' (link de cada objeto
-         de basura). Los nombres deben coincidir con los del mundo. -->
-    <xacro:property name="trash_list"
-      value="trash_can_0 trash_can_1 trash_can_2 trash_crate_0 trash_crate_1 trash_block_0"/>
+         de basura). Los nombres (param trash_list del macro) los pasa el
+         launch y deben coincidir con los modelos de basura inyectados en el
+         mundo. Si trash_list viene vacío no se genera ningún DetachableJoint. -->
     <xacro:macro name="detach_plugin" params="obj">
       <gazebo>
